Commit message: Add gripper joint, arm telemetry

File: arm_ros2_ws/src/arm/description/arm.urdf (robot description, URDF)
Before this commit: robot arm, 8 links, 7 joints
Links:
- added link gripper_dummy
Joints:
- added joint gripper: type revolute, parent wrist_roll_link, child gripper_dummy, origin xyz=-0.046784 0.030841 0.14058 rpy=-0.18325 -0.49709 0.88442, axis 0 1 0, limit lower=-3.14 upper=3.14 effort=20 velocity=1.0

File: arm_ros2_ws/src/arm_moveit_config/config/arm.ros2_control.xacro (robot description, xacro)
@@ -71,4 +71,13 @@
                 <!-- <state_interface name="effort"/> -->
             </joint>
+            <joint name="gripper">
+                <command_interface name="position"/>
+                <command_interface name="velocity"/>
+                <state_interface name="position">
+                  <param name="initial_value">${initial_positions['gripper']}</param>
+                </state_interface>
+                <state_interface name="velocity"/>
+                <!-- <state_interface name="effort"/> -->
+            </joint>
         </ros2_control>
     </xacro:macro>
